File: ESP32-C3_breakout.kicad_sch (KiCad schematic)
At the start: 33 parts, among them IC1 STF202-22T1G, J1 USB4105-GF-A, J2 Conn_01x11_Male, J3 Conn_01x11_Male, SW1 SW_Push, SW2 SW_Push, U1 LD1117S33TR_SOT223, U2 ESP32-C3, Y1 40MHz

Commit message: Update KiCad project files and .gitignore
Parts:
- removed C1: 100n, Capacitor_SMD:C_0603_1608Metric, symbol Device:C
- removed C2: 1u, Capacitor_SMD:C_0603_1608Metric, symbol Device:C
- removed C3: 10u, Capacitor_SMD:C_0603_1608Metric, symbol Device:C
- removed J1: USB4105-GF-A, USB4105-GF-A:GCT_USB4105-GF-A, symbol USB4105-GF-A:USB4105-GF-A
- removed J2, J3: Conn_01x11_Male, Connector_PinHeader_2.54mm:PinHeader_1x11_P2.54mm_Vertical, symbol Connector:Conn_01x11_Male
- removed R2, R3: 5k1, Resistor_SMD:R_0603_1608Metric, symbol Device:R
- removed U1: LD1117S33TR_SOT223, Package_TO_SOT_SMD:SOT-89-3, symbol Regulator_Linear:LD1117S33TR_SOT223
- added C16, C17, C18, C19, C20, C21, C22, C23, C24: 100n, Capacitor_SMD:C_0603_1608Metric, symbol Device:C
- added C25, C26, C27: 10n, Capacitor_SMD:C_0603_1608Metric, symbol Device:C
- added C28: 4.7u, Capacitor_SMD:C_0603_1608Metric, symbol Device:C
- added D10, D11, D12, D13, D14, D15, D16, D17, D18, D19, D2, D20, D21, D22, D23, D24, D25, D3, D4, D5, D6, D7, D8, D9: SK6805, LED_SMD:LED_SK6805_PLCC4_2.4x2.7mm_P1.3mm, symbol LED:SK6805
- added D26, D27: LED, LED_SMD:LED_0603_1608Metric, symbol Device:LED
- added J4: USB_C_Receptacle_USB2.0_16P, Connector_USB:USB_C_Receptacle_HRO_TYPE-C-31-M-12, symbol Connector:USB_C_Receptacle_USB2.0_16P
- added R10, R9: 5.1k, Resistor_SMD:R_0603_1608Metric_Pad0.98x0.95mm_HandSolder, symbol Device:R_US
- added R11: R, LED_SMD:LED_SK6805_PLCC4_2.4x2.7mm_P1.3mm, symbol Device:R
- added R12, R13: 1k, LED_SMD:LED_SK6805_PLCC4_2.4x2.7mm_P1.3mm, symbol Device:R
- added R7: 330, LED_SMD:LED_SK6805_PLCC4_2.4x2.7mm_P1.3mm, symbol Device:R
- added R8: 10K, Resistor_SMD:R_0603_1608Metric_Pad0.98x0.95mm_HandSolder, symbol Device:R_US
- added SW3, SW4, SW5: SW_Push, Package_DFN_QFN:Texas_RVA_VQFN-16-1EP_3.5x3.5mm_P0.5mm_EP2.14x2.14mm_ThermalVias, symbol Switch:SW_Push
- added TP1, TP2: TestPoint, TestPoint:TestPoint_Pad_1.0x1.0mm, symbol Connector:TestPoint
- added U3: TP4056-42-ESOP8, Package_SO:SOIC-8-1EP_3.9x4.9mm_P1.27mm_EP2.41x3.3mm_ThermalVias, symbol Battery_Management:TP4056-42-ESOP8
- added U4: AP2112K-1.2, Package_TO_SOT_SMD:SOT-23-5, symbol Regulator_Linear:AP2112K-1.2
Connections:
- net +3V3: now also C16.2, C17.2, C18.2, C19.2, C20.2, C21.2, C22.2, C23.2, C24.2, D10.4 (VDD), D11.4 (VDD), D12.4 (VDD), D13.4 (VDD), D14.4 (VDD), D15.4 (VDD), D16.4 (VDD), D17.4 (VDD), D18.4 (VDD), D19.4 (VDD), D2.4 (VDD), D20.4 (VDD), D21.4 (VDD), D22.4 (VDD), D23.4 (VDD), D24.4 (VDD), D25.4 (VDD), D3.4 (VDD), D4.4 (VDD), D5.4 (VDD), D6.4 (VDD), D7.4 (VDD), D8.4 (VDD), D9.4 (VDD), U4.5 (VOUT)
- net GND: now also C16.1, C17.1, C18.1, C19.1, C20.1, C21.1, C22.1, C23.1, C24.1, C25.1, C26.1, C27.1, C28.2, D10.2 (VSS), D11.2 (VSS), D12.2 (VSS), D13.2 (VSS), D14.2 (VSS), D15.2 (VSS), D16.2 (VSS), D17.2 (VSS), D18.2 (VSS), D19.2 (VSS), D2.2 (VSS), D20.2 (VSS), D21.2 (VSS), D22.2 (VSS), D23.2 (VSS), D24.2 (VSS), D25.2 (VSS), D3.2 (VSS), D4.2 (VSS), D5.2 (VSS), D6.2 (VSS), D7.2 (VSS), D8.2 (VSS), D9.2 (VSS), J4.A1 (GND), J4.A12 (GND), J4.B1 (GND), J4.B12 (GND), R10.1, R11.2, R8.2, R9.2, SW3.2, SW4.2, SW5.2, TP2.1, U3.1 (TEMP), U3.3 (GND), U3.9 (EPAD), U4.2 (GND)
- net GPIO2: now also C25.2, SW3.1
- net GPIO3: now also C26.2, C27.2, SW4.1, SW5.1
- net GPIO8: now also R7.1
- net USB_+5V: no longer IC1.1 (VBUS)
- net D_N: no longer names the net of IC1.2 (D(IN)_1)
- net D_N: now also J4.A6 (D+), J4.B6 (D+)
- net D_P: no longer names the net of IC1.3 (D(IN)_2)
- net D_P: now also J4.A7 (D-), J4.B7 (D-)
- new net: D18.1 (DOUT), D19.3 (DIN)
- new net: D17.1 (DOUT), D18.3 (DIN)
- new net: D10.1 (DOUT), D11.3 (DIN)
- new net: D10.3 (DIN), D9.1 (DOUT)
- new net: D15.1 (DOUT), D16.3 (DIN)
- new net: D14.1 (DOUT), D15.3 (DIN)
- new net: D16.1 (DOUT), D17.3 (DIN)
- new net: D2.1 (DOUT), D3.3 (DIN)
- new net: D2.3 (DIN), R7.2
- new net: D26.1 (K), R12.2
- new net: C28.1, TP1.1, U3.5 (BAT), U4.1 (VIN), U4.3 (EN)
- new net: D12.1 (DOUT), D13.3 (DIN)
- new net: D11.1 (DOUT), D12.3 (DIN)
- new net: D4.1 (DOUT), D5.3 (DIN)
- new net: D3.1 (DOUT), D4.3 (DIN)
- new net: D23.1 (DOUT), D24.3 (DIN)
- new net: D22.1 (DOUT), D23.3 (DIN)
- new net: D21.1 (DOUT), D22.3 (DIN)
- new net: D19.1 (DOUT), D20.3 (DIN)
- new net: J4.A5 (CC1), R9.1
- new net: D8.1 (DOUT), D9.3 (DIN)
- new net: D26.2 (A), U3.7 (~{CHRG})
- new net: R11.1, U3.2 (PROG)
- new net: D27.2 (A), U3.6 (~{STDBY})
- new net: D24.1 (DOUT), D25.3 (DIN)
- new net: D7.1 (DOUT), D8.3 (DIN)
- new net: D6.1 (DOUT), D7.3 (DIN)
- new net: J4.B5 (CC2), R10.2
- new net: D20.1 (DOUT), D21.3 (DIN)
- new net: D13.1 (DOUT), D14.3 (DIN)
- new net: D27.1 (K), R13.2
- new net: D5.1 (DOUT), D6.3 (DIN)
- new net: J4.S1 (SHIELD), R8.1
- new net VBUS: IC1.1 (VBUS), J4.A4 (VBUS), J4.A9 (VBUS), J4.B4 (VBUS), J4.B9 (VBUS), R12.1, R13.1, U3.4 (V_{CC}), U3.8 (CE)
- no-connect marks 10 -> 11
Other:
- note removed: "3V3 Voltage regulator"
- note removed: "Connectors"
- note removed: "USB-C & ESD protection"
- moved on the sheet: C5
